File: DarkScope-Board/DarkScope.sch (EAGLE design)
At the start: 170 parts, among them IC1 ATSAME70Q21A-AN, IC2 TL084D, IC3 TL084D, IC4 TL084D, IC5 TL084D, IC6 AT45DB161E-SSHD-T, IC7 AT45DB161E-SSHD-T, IC8 MCP73871-2CAI_ML, K1 4-1462037-0 (3V Version), K2 4-1462037-0 (3V Version), K3 4-1462037-0 (3V Version), K4 4-1462037-0 (3V Version), X1 1-227161-0, X2 1-227161-0, X3 1-227161-0, X5 1-227161-0

Commit message: Added Devices and Connections
Added Devices and Connections
Parts:
- removed C10, C18, C19, C27, C28, C36: 0.1uf, rcl:C-EUC0603
- removed C11, C20, C29: 220pf, rcl:C-EUC0603
- removed C12, C21, C30: 3pf, rcl:C-EUC0603
- removed C13, C22, C31: 1PF, rcl:C-EUC0603
- removed C14, C15, C23, C24, C32, C33: 30pf, rcl:C-TRIMM3018_11
- removed C16, C17, C25, C26, C34, C35: 120pf, rcl:C-EUC0603
- removed D2, D3, D4: ss14, diode:SCHOTTKY-DIODESMD
- removed K2, K3, K4: 4-1462037-0 (3V Version), SamacSys_Parts:4-1462037-0
- removed R21, R34, R35, R39, R52, R53, R57, R70, R71: 100k, rcl:R-US_R0603
- removed R22, R40, R58: 1.8M, rcl:R-US_R0603
- removed R23, R41, R59: 2M, rcl:R-US_R0603
- removed R24, R42, R60: 200k, rcl:R-US_R0603
- removed R25, R43, R61: 20k, rcl:R-US_R0603
- removed R26, R44, R62: 300, rcl:R-US_R0603
- removed R27, R45, R63: 180, rcl:R-US_R0603
- removed R28, R32, R33, R46, R50, R51, R64, R68, R69: 120, rcl:R-US_R0603
- removed R29, R36, R47, R54, R65, R72: 1k, rcl:R-US_R0603
- removed R30, R48, R66: 3k, rcl:R-US_R0603
- removed R31, R49, R67: 1.5k, rcl:R-US_R0603
- removed R37, R55: 10M, rcl:R-US_R0603
- removed R38, R56: 1M, rcl:R-US_R0603
- removed T11, T12, T13, T14, T15, T16, T17, T18, T19, T20, T21, T22, T23, T24, T25, T26, T27, T28, T29, T30, T31, T32, T33, T34, T35, T36, T37, T38, T39, T40: (no value), DC_LOAD_AU:BC817-40-NPN-SOT23-BEC
- removed X2, X3, X5: 1-227161-0, con-coax:1-227161-0
- added C37: 100uF Tantalum, rcl:C-USC1206
- added D5, D6: (no value), eagle-ltspice:SCHOTTKY-DIODESMC
- added NTC: 10K, rcl:R-US_R0603
- added PROG1: 2K2, rcl:R-US_R0603
- added PROG2, R74, R75, R76, R77: 10k, rcl:R-US_R0603
- added SD1: ST-TF-003A, Seeed-Connector:MICRO-SD-CARD-SOCKET-9P(ST-TF-003A)
- added T41: (no value), DC_LOAD_AU:BC817-40-NPN-SOT23-BEC
- added U$22, U$23: CY62167DV30LLCY62167DV30LL-55BVI, Boltz_RnD:CY62167DV30LLCY62167DV30LL-55BVI
- added USB1: ZX62-B-5PA, Seeed-Connector:MICRO-USB-SMD(ZX62-B-5PA)
- added VBAT+, VBAT-/GND: (no value), wirepad:SMD5
- IC3: value TL084D -> TLE2082ID; device linear:TL084D -> SamacSys_Parts:TLE2082ID
- IC4, IC5: value TL084D -> SP6641BEK-L-3-3_TR; device linear:TL084D -> SamacSys_Parts:SP6641BEK-L-3-3_TR
- R19: value 10M -> 10E
- R20: value 1M -> 10E
Connections:
- removed net N$100: R62.2, R63.1, T38.C
- removed net N$101: R63.2, R64.1, T39.C
- removed net N$102: T35.B
- removed net N$103: T36.B
- removed net N$104: T37.B
- removed net N$105: T34.B
- removed net N$106: T33.B
- removed net N$107: T32.B
- removed net N$108: IC5C.+IN, T38.E, T39.E, T40.E
- removed net N$109: IC5C.-IN, R65.1, R66.1, R67.2
- removed net N$110: IC5C.OUT, R65.2, R68.1, R69.2
- removed net N$111: C35.1, R68.2
- removed net N$112: IC5D.+IN, R69.1, R70.2
- removed net N$113: IC5D.OUT, R70.1, R72.2
- removed net N$114: C36.1, IC5D.-IN, R71.2
- removed net N$115: R71.1
- removed net N$116: R72.1
- removed net N$32: C10.1, K2.7, R19.1, R20.2, T12.C
- removed net N$33: K2.5, R19.2
- removed net N$34: T11.B
- removed net N$35: C10.2, T13.C
- removed net N$36: C11.1, C12.1, C13.1, R21.2, R22.2, R23.2, T12.E, T13.E, T14.E
- removed net N$37: C11.2, R21.1, T15.C
- removed net N$38: C12.2, C14.E, R22.1, R24.1, T16.C
- removed net N$39: C13.2, C15.E, C16.1, R23.1, R25.1, T17.C
- removed net N$40: IC3B.+IN, T15.E, T16.E, T17.E
- removed net N$41: IC3B.-IN, IC3B.OUT, R26.1, T20.C
- removed net N$42: R26.2, R27.1, T18.C
- removed net N$43: R27.2, R28.1, T19.C
- removed net N$44: T15.B
- removed net N$45: T16.B
- removed net N$46: T17.B
- removed net N$47: T14.B
- removed net N$48: T13.B
- removed net N$49: T12.B
- removed net N$50: IC3C.+IN, T18.E, T19.E, T20.E
- removed net N$51: IC3C.-IN, R29.1, R30.1, R31.2
- removed net N$52: IC3C.OUT, R29.2, R32.1, R33.2
- removed net N$53: C17.1, R32.2
- removed net N$54: IC3D.+IN, R33.1, R34.2
- removed net N$55: IC3D.OUT, R34.1, R36.2
- removed net N$56: C18.1, IC3D.-IN, R35.2
- removed net N$57: R35.1
- removed net N$58: R36.1
- removed net N$59: D3.A, K3.1, T21.C
- removed net N$60: K3.6, X2.1
- removed net N$61: C19.1, K3.7, R37.1, R38.2, T22.C
- removed net N$62: K3.5, R37.2
- removed net N$63: T21.B
- removed net N$64: C19.2, T23.C
- removed net N$65: C20.1, C21.1, C22.1, R39.2, R40.2, R41.2, T22.E, T23.E, T24.E
- removed net N$66: C20.2, R39.1, T25.C
- removed net N$67: C21.2, C23.E, R40.1, R42.1, T26.C
- removed net N$68: C22.2, C24.E, C25.1, R41.1, R43.1, T27.C
- removed net N$69: IC4B.+IN, T25.E, T26.E, T27.E
- removed net N$70: IC4B.-IN, IC4B.OUT, R44.1, T30.C
- removed net N$71: R44.2, R45.1, T28.C
- removed net N$72: R45.2, R46.1, T29.C
- removed net N$73: T25.B
- removed net N$74: T26.B
- removed net N$75: T27.B
- removed net N$76: T24.B
- removed net N$77: T23.B
- removed net N$78: T22.B
- removed net N$79: IC4C.+IN, T28.E, T29.E, T30.E
- removed net N$80: IC4C.-IN, R47.1, R48.1, R49.2
- removed net N$81: IC4C.OUT, R47.2, R50.1, R51.2
- removed net N$82: C26.1, R50.2
- removed net N$83: IC4D.+IN, R51.1, R52.2
- removed net N$84: IC4D.OUT, R52.1, R54.2
- removed net N$85: C27.1, IC4D.-IN, R53.2
- removed net N$86: R53.1
- removed net N$87: R54.1
- removed net N$88: D4.A, K4.1, T31.C
- removed net N$89: K4.6, X3.1
- removed net N$90: C28.1, K4.7, R55.1, R56.2, T32.C
- removed net N$91: K4.5, R55.2
- removed net N$92: T31.B
- removed net N$93: C28.2, T33.C
- removed net N$94: C29.1, C30.1, C31.1, R57.2, R58.2, R59.2, T32.E, T33.E, T34.E
- removed net N$95: C29.2, R57.1, T35.C
- removed net N$96: C30.2, C32.E, R58.1, R60.1, T36.C
- removed net N$97: C31.2, C33.E, C34.1, R59.1, R61.1, T37.C
- removed net N$98: IC5B.+IN, T35.E, T36.E, T37.E
- removed net N$99: IC5B.-IN, IC5B.OUT, R62.1, T40.C
- new net +5V/1: IC3.VCC+, R20.1
- new net 3V3: T41.E
- new net 3V3D: T41.C
- new net BMC_PG: R76.1
- new net BMC_STAT1: R74.1
- new net BMC_STAT2: R75.1
- new net CNTRL_3_3V: T41.B
- new net N$117: IC8.STAT1/!LBO, R74.2
- new net N$118: IC8.THERM, NTC.2
- new net N$119: IC8.!PG, R76.2
- new net N$120: IC8.STAT2, R75.2
- new net N$121: IC8.PROG1, PROG1.2
- new net N$122: IC8.VBAT, IC8.VBAT_1, IC8.VBAT_SENSE, VBAT+.P
- new net N$123: IC8.PROG2, PROG2.1
- new net N$124: IC8.CE, R77.1
- new net N$125: IC8.EP, IC8.OUT
- new net USBD+: USB1.D+
- new net USBD-: USB1.D-
- new net USBID: USB1.ID
- new net VBUS: D5.C, D6.C, USB1.VBUS
- net +5V: now also C37.1, D5.A, D6.A, IC8.IN, IC8.IN_1, IC8.VPCC, PROG2.2, R77.2; no longer R30.2, R48.2, R66.2
- net +5V/2: now also R19.1; no longer D2.C, D3.C, D4.C, K2.8, K3.8, K4.8
- net GND: now also C37.2, IC3.VCC-, IC8.VSS, IC8.VSS_1, PROG1.1, USB1.GND, USB1.SHIELD, VBAT-/GND.P; no longer C14.A, C15.A, C16.2, C17.2, C18.2, C23.A, C24.A, C25.2, C26.2, C27.2, C32.A, C33.A, C34.2, C35.2, C36.2, R20.1, R24.2, R25.2, R28.2, R31.1, R38.1, R42.2, R43.2, R46.2, R49.1, R56.1, R60.2, R61.2, R64.2, R67.1, T11.E, T14.C, T21.E, T24.C, T31.E, T34.C, X2.2, X3.2, X5.2
- net N$13: now also IC3.1IN+; no longer IC2B.+IN
- net N$14: now also IC5.VOUT, R19.2; no longer IC2B.-IN, IC2B.OUT, R8.1, T10.C
- net N$21: now also IC3.2IN+; no longer IC2C.+IN
- net N$22: now also IC3.2IN-; no longer IC2C.-IN
- net N$23: now also IC3.2OUT; no longer IC2C.OUT
- net N$30: now also IC3.1IN-, IC3.1OUT, R8.1, T10.C; no longer D2.A, K2.1, T11.C
- net N$31: now also IC4.VOUT, R20.2; no longer K2.6, X5.1
Other:
- note added: "3.3V Peripheral Power Control"
- note added: "Li-Ion Battery"
- note added: "MicroUSB (For Charging and Data Transfer)"
- note added: "Power Supply and Input Regulation"
- note removed: "Power Supply"
- note removed: "Probe Channel 2"
- note removed: "Probe Channel 3"
- note removed: "Probe Channel 4"
- note removed: "USB and Charging Circuitry"

Commit message: Added Components and Modified Conections
Updated The OP-amps and BJTs and modified connections.
Parts:
- removed D1: ss14, diode:SCHOTTKY-DIODESMD
- removed IC2: TL084D, linear:TL084D
- removed K1: 4-1462037-0 (3V Version), SamacSys_Parts:4-1462037-0
- added C10, C12: 100uf, resistor:C-USC0603K
- added C11, C13: 1uf, resistor:C-USC0603K
- added C14, C15: (no value), rcl:C-USC0603K
- added D2, D3: ss14, diode:SCHOTTKY-DIODESMC
- added D7: 3V3_Z_D, diode:ZENER-DIODESOD80C
- added IC10: REG1117, burr-brown:REG1117
- added IC9: TLE2082ID, SamacSys_Parts:TLE2082ID
- added IC_VDD_SELECT, JMP1: 0R-JUMPC, jump-0r-smd:0R-JUMPC
- added L1, L2: 10uH, eagle-ltspice:L0204/7
- added R21: 680E, rcl:R-US_R0603
- added R22: 10K, rcl:R-US_R0603
- added R23: 68K, rcl:R-US_R0603
- added SJ1: (no value), jumper:SJ
- added TP1, TP10, TP11, TP12, TP13, TP14, TP15, TP16, TP17, TP18, TP19, TP2, TP20, TP21, TP22, TP23, TP24, TP25, TP26, TP27, TP28, TP29, TP3, TP30, TP31, TP32, TP4, TP5, TP6, TP7, TP8, TP9: TPTP07R, testpad:TPTP07R
- IC4, IC5: value SP6641BEK-L-3-3_TR -> SP6641BEK-L-5-0
- R1: value 10M -> 22K
- R13: value 1.5k -> 2.2K
- R14: value 120 -> 330E
- R2: value 1M -> 10K
- T1, T10, T2, T3, T4, T41, T5, T6, T7, T8, T9: value (none) -> BC807-40SMD; device DC_LOAD_AU:BC817-40-NPN-SOT23-BEC -> transistor-pnp:BC807-40SMD
Connections:
- removed net N$125: IC8.EP, IC8.OUT
- removed net N$4 (its old number): K1.6, X1.1
- new net +3V3: C10.1, IC4.VBATT, IC_VDD_SELECT-0R.1, L1.2
- new net N$14: D2.A, IC4.LX, L1.1
- new net N$2: JMP1-0R.1, R1.1, R2.2, TP12.TP
- new net N$33: D3.A, IC5.LX, L2.1
- new net N$34: R13.1, R21.2, SJ1.2
- new net N$35: T8.B
- new net N$36: R22.2, T1.E
- new net N$37: R1.2, R23.1
- new net N$38: JMP1-0R.2, T1.C
- new net N$39: T9.B
- new net VCC: C12.1, C14.1, IC10.VIN, IC5.VBATT, IC8.OUT, IC8.OUT_1, L2.2, TP30.TP
- new net VCCINT: IC_VDD_SELECT-0R.2
- net +5V: now also TP17.TP, TP25.TP; no longer R12.2
- net +5V/1: now also C11.1, D2.C, IC9.VCC+, IC_VDD_SELECT-0R.3, R12.2, TP11.TP, TP28.TP, TP7.TP
- net +5V/2: now also C13.1, D3.C, TP27.TP; no longer D1.C, K1.8
- net 3V3: now also TP31.TP
- net 3V3D: now also C15.1, IC10.VOUT, TP29.TP, TP32.TP
- net BMC_PG: now also TP19.TP
- net BMC_STAT1: now also TP21.TP
- net BMC_STAT2: now also TP20.TP
- net GND: now also C10.2, C11.2, C12.2, C13.2, C14.2, C15.2, D7.A, IC10.GND, IC4.GND, IC5.GND, IC9.VCC-, R21.1, SJ1.1, TP15.TP, TP26.TP; no longer R13.1, R2.1, T1.E, X1.2
- net N$1: now also R2.1, X1.2; no longer D1.A, K1.1, T1.C
- net N$118: now also TP18.TP
- net N$121: now also TP16.TP
- net N$122: now also TP14.TP
- net N$13: now also TP3.TP
- net N$21: now also TP4.TP
- net N$24: now also TP8.TP
- net N$25: now also IC9.1IN+; no longer IC2D.+IN
- net N$26: now also IC9.1OUT, TP6.TP; no longer IC2D.OUT
- net N$27: now also IC9.1IN-; no longer IC2D.-IN
- net N$28: now also TP10.TP
- net N$29: now also TP9.TP
- net N$30: now also D7.C, TP5.TP
- net N$6: now also R22.1, R23.2, TP1.TP, TP13.TP, X1.1; no longer K1.7, R1.1, R2.2
- net N$7: now also T10.B; no longer K1.5, R1.2
- net N$8: now also TP2.TP
- net USBD+: now also TP23.TP
- net USBD-: now also TP24.TP
- net USBID: now also TP22.TP
Other:
- note added: "3V3 Regulator Circuit"
- note added: "5V Power for ICs"
- note added: "5V Power for Relays and Power Electronics"
- note added: "Changing the value of resistor R13 & R21 to 2.880K (2.2K + 680E) will toggle the 5V Peak output to 3V3 Peak .For 5V Levels the value is 1.5K(1.5K + Shorted SJ1)"
- note added: "VINT Voltage Source Selection"

Commit message: Updated Files and Timeline
Updated the timeline for product completetion, and backed up last saved work.
Parts:
- added D1, D4: (no value), diode:ZENER-DIODESOD80C
- added R24, R25, R26, R27: 1k, rcl:R-US_R0603
- added T11, T12: BC807-40SMD, transistor-pnp:BC807-40SMD
Connections:
- new net N$40: D1.A, R24.2, R25.2
- new net N$41: R25.1, T11.B
- new net N$42: D1.C, T11.C
- new net N$43: D4.A, R26.2, R27.2
- new net N$44: R27.1, T12.B
- new net N$46: C1.1, T12.E, T2.C
- net N$6: now also D4.C, T12.C; no longer C1.1, T2.C
Other:
- moved on the sheet: JMP1-0R, R1, R2, R22, R23, T1, TP12, TP13
