File: Hardware/DarkScope-Board/BaseBoard.sch (EAGLE design)
At the start: 17 parts, among them U1 STM32F103CBT6

Commit message: CP PSU
Parts:
- added C10, C12, C14, C15, C9: 100uF, rcl:CPOL-USCT6032
- added C11, C13: 0.1u, rcl:C-EUC1206
- added D1: SS14, diode:ES2D
- added D2: 1N5819-B, diode:1N5819-B
- added IC1: 7805DT, linear:7805DT
- added IC2: REG1117, burr-brown:REG1117
- added IC3: 7905, linear:79L05Z
- added J1: DCJ0202, con-jack:DCJ0202
- added JMP1, JMP2: 0R-JUMPC, jump-0r-smd:0R-JUMPC
- added L2, L3: 100uH, rcl:L-US0204/5
- added LED1: (no value), led:LEDCHIPLED_1206
- added R2, R3, R4, R5, R6, R7, R8: 470R, rcl:R-US_R0805
- added SJ3: (no value), jumper:SJW
- added T1: (no value), transistor:-PNP-TO92
- added T2: (no value), transistor:-NPN-TO92
- added TP10, TP11, TP12, TP13, TP3, TP4, TP5, TP6, TP7, TP8, TP9: TPB1,27, testpad:TPB1,27
- added X1, X2: TSW-102-07-G-S, con-samtec:TSW-102-07-G-S
- L1: value (none) -> 100uH
- Q1: value (none) -> 8MHz
Connections:
- removed net N$25: C7.2, C8.2
- new net +12V: D1.A, J1.1, R3.1, T1.E, X2-2.1
- new net +5V: C10.+, JMP1-0R.3, L2.2, SJ3.2, TP4.TP
- new net N$10: C13.2, R6.2
- new net N$11: D2.C, T1.C
- new net N$12: C14.+, D2.A, L3.1
- new net N$13: C15.+, IC3.VI, L3.2, R8.2, TP12.TP
- new net N$14: IC3.VO, TP13.TP
- new net N$15: R7.1, R8.1
- new net N$2: LED1.A, R2.2
- new net N$3: C11.1, IC1.VO, JMP1-0R.1, L2.1, SJ3.1
- new net N$4: R3.2, R4.2, T1.B
- new net N$5: C12.+, IC2.VOUT, JMP2-0R.1, TP5.TP
- new net N$6: R4.1, T2.C
- new net N$7: C13.1, R5.2, T2.B
- new net N$8: C9.+, D1.C, IC1.VI, TP3.TP
- new net N$9: IC2.VIN, JMP1-0R.2, TP7.TP
- net +3V3: now also JMP2-0R.2, R2.1, TP6.TP
- net DB2: now also X1-1.1
- net GND: now also C10.-, C11.2, C12.-, C14.-, C15.-, C7.2, C8.2, C9.-, IC1.GND, IC2.GND, IC3.GND, J1.3, R5.1, T2.E, TP10.TP, TP11.TP, TP8.TP, TP9.TP, U1.VSSA, X1-2.1, X2-1.1
- net LED: now also LED1.C
Other:
- note added: "MCU"
- note added: "PSU"

Commit message: CP PSU Completed
Parts:
- added L4: 1mH/1A, rcl:L-US6000-XXX-RC
- added TP14, TP15: TPB1,27, testpad:TPB1,27
- R3, R5, R8: value 470R -> 10K
- R4: value 470R -> 1.5K
- R7: value 470R -> 1K
- T2: value (none) -> 9014
Connections:
- net N$14 renamed -5V
- removed net N$15: R7.1, R8.1
- net +3V3: now also R7.2
- net GND: now also L4.2, TP14.TP, TP15.TP
- net N$11: now also L4.1
- net V-MON: now also R7.1, R8.1
- net VGEN: now also R6.1
Changed lines of the file:
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@@
 <part name="P+3" library="supply1" library_urn="urn:adsk.eagle:library:371" deviceset="+12V" device=""/>
 <part name="T1" library="transistor" library_urn="urn:adsk.eagle:library:402" deviceset="*-PNP-" device="TO92" package3d_urn="urn:adsk.eagle:package:28523/2"/>
-<part name="R3" library="rcl" library_urn="urn:adsk.eagle:library:334" deviceset="R-US_" device="R0805" package3d_urn="urn:adsk.eagle:package:23553/2" value="470R"/>
-<part name="R4" library="rcl" library_urn="urn:adsk.eagle:library:334" deviceset="R-US_" device="R0805" package3d_urn="urn:adsk.eagle:package:23553/2" value="470R"/>
-<part name="T2" library="transistor" library_urn="urn:adsk.eagle:library:402" deviceset="*-NPN-" device="TO92" package3d_urn="urn:adsk.eagle:package:28523/2"/>
-<part name="R5" library="rcl" library_urn="urn:adsk.eagle:library:334" deviceset="R-US_" device="R0805" package3d_urn="urn:adsk.eagle:package:23553/2" value="470R"/>
+<part name="R3" library="rcl" library_urn="urn:adsk.eagle:library:334" deviceset="R-US_" device="R0805" package3d_urn="urn:adsk.eagle:package:23553/2" value="10K"/>
+<part name="R4" library="rcl" library_urn="urn:adsk.eagle:library:334" deviceset="R-US_" device="R0805" package3d_urn="urn:adsk.eagle:package:23553/2" value="1.5K"/>
+<part name="T2" library="transistor" library_urn="urn:adsk.eagle:library:402" deviceset="*-NPN-" device="TO92" package3d_urn="urn:adsk.eagle:package:28523/2" value="9014"/>
+<part name="R5" library="rcl" library_urn="urn:adsk.eagle:library:334" deviceset="R-US_" device="R0805" package3d_urn="urn:adsk.eagle:package:23553/2" value="10K"/>
 <part name="R6" library="rcl" library_urn="urn:adsk.eagle:library:334" deviceset="R-US_" device="R0805" package3d_urn="urn:adsk.eagle:package:23553/2" value="470R"/>
 <part name="C13" library="rcl" library_urn="urn:adsk.eagle:library:334" deviceset="C-EU" device="C1206" package3d_urn="urn:adsk.eagle:package:23618/2" value="0.1u"/>
@@
 <part name="TP13" library="testpad" library_urn="urn:adsk.eagle:library:385" deviceset="TP" device="B1,27" package3d_urn="urn:adsk.eagle:package:27944/2"/>
 <part name="GND22" library="supply1" library_urn="urn:adsk.eagle:library:371" deviceset="GND" device=""/>
-<part name="R7" library="rcl" library_urn="urn:adsk.eagle:library:334" deviceset="R-US_" device="R0805" package3d_urn="urn:adsk.eagle:package:23553/2" value="470R"/>
-<part name="R8" library="rcl" library_urn="urn:adsk.eagle:library:334" deviceset="R-US_" device="R0805" package3d_urn="urn:adsk.eagle:package:23553/2" value="470R"/>
+<part name="R7" library="rcl" library_urn="urn:adsk.eagle:library:334" deviceset="R-US_" device="R0805" package3d_urn="urn:adsk.eagle:package:23553/2" value="1K"/>
+<part name="R8" library="rcl" library_urn="urn:adsk.eagle:library:334" deviceset="R-US_" device="R0805" package3d_urn="urn:adsk.eagle:package:23553/2" value="10K"/>
+<part name="+3V6" library="supply1" library_urn="urn:adsk.eagle:library:371" deviceset="+3V3" device=""/>
+<part name="P-1" library="supply1" library_urn="urn:adsk.eagle:library:371" deviceset="-5V" device=""/>
+<part name="L4" library="rcl" library_urn="urn:adsk.eagle:library:334" deviceset="L-US" device="6000-XXX-RC" package3d_urn="urn:adsk.eagle:package:23538/1" value="1mH/1A"/>
+<part name="GND23" library="supply1" library_urn="urn:adsk.eagle:library:371" deviceset="GND" device=""/>
+<part name="TP14" library="testpad" library_urn="urn:adsk.eagle:library:385" deviceset="TP" device="B1,27" package3d_urn="urn:adsk.eagle:package:27944/2"/>
+<part name="TP15" library="testpad" library_urn="urn:adsk.eagle:library:385" deviceset="TP" device="B1,27" package3d_urn="urn:adsk.eagle:package:27944/2"/>
+<part name="GND24" library="supply1" library_urn="urn:adsk.eagle:library:371" deviceset="GND" device=""/>
+<part name="GND25" library="supply1" library_urn="urn:adsk.eagle:library:371" deviceset="GND" device=""/>
 </parts>
 <sheets>
@@
 <sheet>
 <plain>
-<text x="11.43" y="95.25" size="1.778" layer="91">PSU</text>
+<text x="6.35" y="128.27" size="1.778" layer="91">PSU</text>
 </plain>
 <instances>
@@
 <attribute name="NAME" x="274.32" y="79.7814" size="1.778" layer="95" rot="R180"/>
 <attribute name="VALUE" x="274.32" y="84.582" size="1.778" layer="96" rot="R180"/>
+</instance>
+<instance part="+3V6" gate="G$1" x="259.08" y="73.66" smashed="yes" rot="R90">
+<attribute name="VALUE" x="264.16" y="71.12" size="1.778" layer="96" rot="R180"/>
+</instance>
+<instance part="P-1" gate="1" x="295.91" y="110.49" smashed="yes" rot="R90">
+<attribute name="VALUE" x="298.45" y="107.95" size="1.778" layer="96" rot="R180"/>
+</instance>
+<instance part="L4" gate="G$1" x="212.09" y="100.33" smashed="yes">
+<attribute name="NAME" x="210.82" y="95.25" size="1.778" layer="95" rot="R90"/>
+<attribute name="VALUE" x="215.9" y="95.25" size="1.778" layer="96" rot="R90"/>
+</instance>
+<instance part="GND23" gate="1" x="212.09" y="90.17" smashed="yes">
+<attribute name="VALUE" x="209.55" y="87.63" size="1.778" layer="96"/>
+</instance>
+<instance part="TP14" gate="G$1" x="292.1" y="74.93" smashed="yes">
+<attribute name="NAME" x="290.83" y="76.2" size="1.778" layer="95"/>
+<attribute name="TP_SIGNAL_NAME" x="293.37" y="73.66" size="1.778" layer="97"/>
+</instance>
+<instance part="TP15" gate="G$1" x="299.72" y="74.93" smashed="yes">
+<attribute name="NAME" x="298.45" y="76.2" size="1.778" layer="95"/>
+<attribute name="TP_SIGNAL_NAME" x="300.99" y="73.66" size="1.778" layer="97"/>
+</instance>
+<instance part="GND24" gate="1" x="292.1" y="69.85" smashed="yes">
+<attribute name="VALUE" x="289.56" y="67.31" size="1.778" layer="96"/>
+</instance>
+<instance part="GND25" gate="1" x="299.72" y="69.85" smashed="yes">
+<attribute name="VALUE" x="297.18" y="67.31" size="1.778" layer="96"/>
 </instance>
 </instances>
@@
 <wire x1="115.57" y1="95.25" x2="115.57" y2="100.33" width="0.1524" layer="91"/>
 </segment>
+<segment>
+<pinref part="+3V6" gate="G$1" pin="+3V3"/>
+<pinref part="R7" gate="G$1" pin="2"/>
+<wire x1="261.62" y1="73.66" x2="265.43" y2="73.66" width="0.1524" layer="91"/>
+</segment>
 </net>
 <net name="N$8" class="0">
@@
 <pinref part="IC3" gate="A1" pin="GND"/>
 <wire x1="270.51" y1="96.52" x2="270.51" y2="102.87" width="0.1524" layer="91"/>
+</segment>
+<segment>
+<pinref part="GND23" gate="1" pin="GND"/>
+<pinref part="L4" gate="G$1" pin="2"/>
+</segment>
+<segment>
+<pinref part="GND24" gate="1" pin="GND"/>
+<pinref part="TP14" gate="G$1" pin="TP"/>
+</segment>
+<segment>
+<pinref part="GND25" gate="1" pin="GND"/>
+<pinref part="TP15" gate="G$1" pin="TP"/>
 </segment>
 </net>
@@
 <pinref part="T1" gate="G$1" pin="C"/>
 <pinref part="D2" gate="G$1" pin="C"/>
-<wire x1="205.74" y1="110.49" x2="218.44" y2="110.49" width="0.1524" layer="91"/>
+<wire x1="205.74" y1="110.49" x2="212.09" y2="110.49" width="0.1524" layer="91"/>
+<pinref part="L4" gate="G$1" pin="1"/>
+<wire x1="212.09" y1="110.49" x2="218.44" y2="110.49" width="0.1524" layer="91"/>
+<wire x1="212.09" y1="107.95" x2="212.09" y2="110.49" width="0.1524" layer="91"/>
+<junction x="212.09" y="110.49"/>
 </segment>
 </net>
@@
 </segment>
 </net>
-<net name="N$14" class="0">
+<net name="-5V" class="0">
 <segment>
 <pinref part="IC3" gate="A1" pin="VO"/>
 <pinref part="TP13" gate="G$1" pin="TP"/>
-<wire x1="288.29" y1="110.49" x2="280.67" y2="110.49" width="0.1524" layer="91"/>
-</segment>
-</net>
-<net name="N$15" class="0">
+<wire x1="293.37" y1="110.49" x2="280.67" y2="110.49" width="0.1524" layer="91"/>
+<pinref part="P-1" gate="1" pin="-5V"/>
+<junction x="293.37" y="110.49"/>
+<wire x1="293.37" y1="110.49" x2="288.29" y2="110.49" width="0.1524" layer="91"/>
+</segment>
+</net>
+<net name="V-MON" class="0">
 <segment>
 <pinref part="R8" gate="G$1" pin="1"/>
@@
 <wire x1="281.94" y1="73.66" x2="281.94" y2="81.28" width="0.1524" layer="91"/>
 <junction x="281.94" y="81.28"/>
-</segment>
-</net>
+<label x="284.48" y="81.28" size="1.778" layer="95"/>
+</segment>
+</net>
+<net name="VGEN" class="0">
+<segment>
+<pinref part="R6" gate="G$1" pin="1"/>
+<wire x1="242.57" y1="73.66" x2="250.19" y2="73.66" width="0.1524" layer="91"/>
+<label x="246.38" y="73.66" size="1.778" layer="95"/>
+</segment>
+</net>

Commit message: Added LCD Header
Parts:
- added JMP3: 0R-JUMPC, jump-0r-smd:0R-JUMPC
- added JP1, JP2: (no value), pinhead:PINHD-1X2
- added LCDHEADER: (no value), con-lstb:MA20-2
- added R9: 180E, rcl:R-US_R0805
- added SJ4, SJ5: (no value), jumper:SJ
Connections:
- removed net N$8: C9.+, D1.C, IC1.VI, TP3.TP
- new net IM0: LCDHEADER.11, SJ4.2
- new net IM3: LCDHEADER.21, SJ5.1
- new net LED-A: LCDHEADER.16, R9.2
- new net LED-K1: LCDHEADER.15
- new net N$14: LCDHEADER.2
- new net N$15: LCDHEADER.4
- new net N$16: JMP3-0R.2, R9.1
- new net N$17: D1.A, J1.1, X2-2.1
- new net N$19: LCDHEADER.12
- new net N$20: LCDHEADER.14
- new net N$28: LCDHEADER.22
- new net N$35: LCDHEADER.36
- new net N$36: LCDHEADER.38
- new net N$37: LCDHEADER.40
- new net N$38: LCDHEADER.1
- new net N$39: LCDHEADER.3
- new net N$44: LCDHEADER.13
- new net N$55: LCDHEADER.35
- new net N$56: LCDHEADER.37
- new net N$57: LCDHEADER.39
- net +12V: now also C9.+, D1.C, IC1.VI, JMP3-0R.3, TP3.TP; no longer D1.A, J1.1, X2-2.1
- net +3V3: now also LCDHEADER.32, LCDHEADER.33, LCDHEADER.6, SJ4.1
- net +5V: now also JMP3-0R.1
- net DB0: now also LCDHEADER.23
- net DB1: now also LCDHEADER.24
- net DB2: now also LCDHEADER.25
- net DB3: now also LCDHEADER.26
- net DB4: now also LCDHEADER.27
- net DB5: now also LCDHEADER.28
- net DB6: now also LCDHEADER.29
- net DB7: now also LCDHEADER.30
- net GND: now also LCDHEADER.17, LCDHEADER.18, LCDHEADER.19, LCDHEADER.20, LCDHEADER.34, LCDHEADER.5, SJ5.2
- net LCD_NCS: now also LCDHEADER.7
- net LCD_NRD: now also LCDHEADER.10
- net LCD_NRESET: now also LCDHEADER.31
- net LCD_NWR: now also LCDHEADER.9
- net LCD_RS: now also LCDHEADER.8
Other:
- note added: "LCD Section"

Commit message: DP
Parts:
- added JP3: (no value), pinhead:PINHD-1X4
- added JP4: (no value), pinhead:PINHD-1X2
- added JP5: (no value), pinhead:PINHD-1X3
- added JP6: (no value), pinhead:PINHD-1X12
- added R10, R11, R12: 1K, rcl:R-US_R0805
- added R13, R14: 10K, rcl:R-US_R0805
- added R15, R16: 22E, rcl:R-US_R0805
- added R17: 1.5K, rcl:R-US_R0805
- added TP16, TP17, TP18, TP19, TP20: TPB1,27, testpad:TPB1,27
- added X3: MINI-USB-32005-301, con-cypressindustries:MINI-USB-32005-301
- added X4: 2540-5, con-3m:2540-5
Connections:
- removed net N$24: C6.1, S1.S, S1.S1, U1.NRST
- new net N$18: JP5.3, R11.2
- new net N$25: JP4.1, JP4.2, R12.2
- new net N$26: R17.2, TP18.TP, X3.1
- new net N$27: R16.2, R17.1, X3.3
- new net N$29: R15.2, X3.2
- new net N$41: JP6.10
- new net N$42: JP6.11
- new net N$8: JP5.2, R10.2
- new net NRST: C6.1, JP6.8, S1.S, S1.S1, U1.NRST
- net +3V3: now also JP3.1, JP6.6, JP6.7, R14.1, X4-1.KL, X4-2.KL
- net +5V: now also X4-3.KL, X4-4.KL
- net -5V: now also X4-5.KL, X4-6.KL
- net ADCIN: now also X4-15.KL
- net BTN1: now also JP6.2
- net BTN2: now also JP6.3
- net BTN3: now also JP6.4
- net BTN4: now also JP6.5
- net GND: now also JP3.4, JP5.1, JP6.1, JP6.12, R13.1, X3.5, X4-37.KL, X4-38.KL, X4-39.KL, X4-40.KL
- net LED: now also JP6.9
- net RX1: now also R10.1, TP17.TP
- net SWCLK: now also JP3.3, R13.2
- net SWDIO: now also JP3.2, R14.2
- net TESTSIG: now also R12.1
- net TX1: now also R11.1, TP16.TP
- net USBDM: now also R15.1, TP19.TP
- net USBDP: now also R16.1, TP20.TP
Other:
- note added: "Expansion Port - Analog/Digital Channels"
- note added: "Expansion Port- Buttons"
- note added: "SWD"
- note added: "SWD, Test, USB, and UART"
- note added: "Test Signal Terminal"
- note added: "UART"

Commit message: BaseBoard Schematic Complete
Connections:
- net ADCIN2: now also X4-11.KL
- net ADCIN3: now also X4-10.KL
- net CPLSEL: now also X4-12.KL
- net DB3: now also X4-16.KL
- net DB4: now also X4-17.KL
- net DB5: now also X4-18.KL
- net DB6: now also X4-19.KL
- net DB7: now also X4-20.KL
- net RX1: now also X4-24.KL
- net SWCLK: now also X4-26.KL
- net SWDIO: now also X4-25.KL
- net TESTSIG: now also X4-8.KL
- net TL_PWM: now also X4-21.KL
- net TRIG: now also X4-7.KL
- net TX1: now also X4-23.KL
- net V-MON: now also X4-9.KL
- net VGEN: now also X4-22.KL
- net VSENSEL1: now also X4-13.KL
- net VSENSEL2: now also X4-14.KL
Changed lines of the file:
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@@
 <segment>
 <pinref part="X4" gate="-15" pin="KL"/>
-<wire x1="38.1" y1="53.34" x2="66.04" y2="53.34" width="0.1524" layer="91"/>
-<label x="60.96" y="53.34" size="1.778" layer="95"/>
+<wire x1="38.1" y1="53.34" x2="64.77" y2="53.34" width="0.1524" layer="91"/>
+<label x="67.31" y="53.34" size="1.778" layer="95"/>
 </segment>
 </net>
+<net name="VSENSEL2" class="0">
+<segment>
+<wire x1="64.77" y1="55.88" x2="38.1" y2="55.88" width="0.1524" layer="91"/>
+<label x="78.74" y="57.15" size="1.778" layer="95" rot="R180"/>
+<pinref part="X4" gate="-14" pin="KL"/>
+</segment>
+</net>
+<net name="VSENSEL1" class="0">
+<segment>
+<wire x1="64.77" y1="58.42" x2="38.1" y2="58.42" width="0.1524" layer="91"/>
+<label x="78.74" y="59.69" size="1.778" layer="95" rot="R180"/>
+<pinref part="X4" gate="-13" pin="KL"/>
+</segment>
+</net>
+<net name="CPLSEL" class="0">
+<segment>
+<wire x1="64.77" y1="60.96" x2="38.1" y2="60.96" width="0.1524" layer="91"/>
+<label x="74.93" y="62.23" size="1.778" layer="95" rot="R180"/>
+<pinref part="X4" gate="-12" pin="KL"/>
+</segment>
+</net>
+<net name="ADCIN2" class="0">
+<segment>
+<wire x1="64.77" y1="63.5" x2="38.1" y2="63.5" width="0.1524" layer="91"/>
+<label x="74.93" y="64.77" size="1.778" layer="95" rot="R180"/>
+<pinref part="X4" gate="-11" pin="KL"/>
+</segment>
+</net>
+<net name="ADCIN3" class="0">
+<segment>
+<wire x1="64.77" y1="66.04" x2="38.1" y2="66.04" width="0.1524" layer="91"/>
+<label x="74.93" y="67.31" size="1.778" layer="95" rot="R180"/>
+<pinref part="X4" gate="-10" pin="KL"/>
+</segment>
+</net>
+<net name="V-MON" class="0">
+<segment>
+<wire x1="64.77" y1="68.58" x2="38.1" y2="68.58" width="0.1524" layer="91"/>
+<label x="73.66" y="69.85" size="1.778" layer="95" rot="R180"/>
+<pinref part="X4" gate="-9" pin="KL"/>
+</segment>
+</net>
+<net name="TESTSIG" class="0">
+<segment>
+<wire x1="64.77" y1="71.12" x2="38.1" y2="71.12" width="0.1524" layer="91"/>
+<label x="76.2" y="72.39" size="1.778" layer="95" rot="R180"/>
+<pinref part="X4" gate="-8" pin="KL"/>
+</segment>
+</net>
+<net name="TRIG" class="0">
+<segment>
+<wire x1="64.77" y1="73.66" x2="38.1" y2="73.66" width="0.1524" layer="91"/>
+<label x="71.12" y="74.93" size="1.778" layer="95" rot="R180"/>
+<pinref part="X4" gate="-7" pin="KL"/>
+</segment>
+</net>
+<net name="DB3" class="0">
+<segment>
+<wire x1="38.1" y1="50.8" x2="64.77" y2="50.8" width="0.1524" layer="91"/>
+<label x="67.31" y="50.8" size="1.778" layer="95"/>
+<pinref part="X4" gate="-16" pin="KL"/>
+</segment>
+</net>
+<net name="DB4" class="0">
+<segment>
+<wire x1="38.1" y1="48.26" x2="64.77" y2="48.26" width="0.1524" layer="91"/>
+<label x="67.31" y="48.26" size="1.778" layer="95"/>
+<pinref part="X4" gate="-17" pin="KL"/>
+</segment>
+</net>
+<net name="DB5" class="0">
+<segment>
+<wire x1="38.1" y1="45.72" x2="64.77" y2="45.72" width="0.1524" layer="91"/>
+<label x="67.31" y="45.72" size="1.778" layer="95"/>
+<pinref part="X4" gate="-18" pin="KL"/>
+</segment>
+</net>
+<net name="DB6" class="0">
+<segment>
+<wire x1="38.1" y1="43.18" x2="64.77" y2="43.18" width="0.1524" layer="91"/>
+<label x="67.31" y="43.18" size="1.778" layer="95"/>
+<pinref part="X4" gate="-19" pin="KL"/>
+</segment>
+</net>
+<net name="DB7" class="0">
+<segment>
+<wire x1="38.1" y1="40.64" x2="64.77" y2="40.64" width="0.1524" layer="91"/>
+<label x="67.31" y="40.64" size="1.778" layer="95"/>
+<pinref part="X4" gate="-20" pin="KL"/>
+</segment>
+</net>
+<net name="TL_PWM" class="0">
+<segment>
+<wire x1="38.1" y1="38.1" x2="64.77" y2="38.1" width="0.1524" layer="91"/>
+<label x="67.31" y="38.1" size="1.778" layer="95"/>
+<pinref part="X4" gate="-21" pin="KL"/>
+</segment>
+</net>
+<net name="VGEN" class="0">
+<segment>
+<wire x1="38.1" y1="35.56" x2="64.77" y2="35.56" width="0.1524" layer="91"/>
+<label x="67.31" y="35.56" size="1.778" layer="95"/>
+<pinref part="X4" gate="-22" pin="KL"/>
+</segment>
+</net>
+<net name="TX1" class="0">
+<segment>
+<pinref part="X4" gate="-23" pin="KL"/>
+<wire x1="38.1" y1="33.02" x2="64.77" y2="33.02" width="0.1524" layer="91"/>
+<label x="67.31" y="33.02" size="1.778" layer="95"/>
+</segment>
+</net>
+<net name="RX1" class="0">
+<segment>
+<pinref part="X4" gate="-24" pin="KL"/>
+<wire x1="38.1" y1="30.48" x2="64.77" y2="30.48" width="0.1524" layer="91"/>
+<label x="67.31" y="30.48" size="1.778" layer="95"/>
+</segment>
+</net>
+<net name="SWDIO" class="0">
+<segment>
+<pinref part="X4" gate="-25" pin="KL"/>
+<wire x1="38.1" y1="27.94" x2="64.77" y2="27.94" width="0.1524" layer="91"/>
+<label x="67.31" y="27.94" size="1.778" layer="95"/>
+</segment>
+</net>
+<net name="SWCLK" class="0">
+<segment>
+<pinref part="X4" gate="-26" pin="KL"/>
+<wire x1="38.1" y1="25.4" x2="64.77" y2="25.4" width="0.1524" layer="91"/>
+<label x="67.31" y="25.4" size="1.778" layer="95"/>
+</segment>
+</net>

Commit message: DP
Connections:
- new net VSENSEL3: X4-24.KL
- new net VSENSEL4: X4-25.KL
- net ADCIN: now also X4-23.KL; no longer X4-15.KL
- net ADCIN2: now also X4-27.KL; no longer X4-11.KL
- net ADCIN3: now also X4-28.KL; no longer X4-10.KL
- net BTN1: now also X4-22.KL
- net BTN2: now also X4-21.KL
- net BTN3: now also X4-20.KL
- net BTN4: now also X4-19.KL
- net CPLSEL: now also X4-26.KL; no longer X4-12.KL
- net DB0: now also X4-7.KL
- net DB1: now also X4-8.KL
- net DB2: now also X4-9.KL
- net DB3: now also X4-10.KL; no longer X4-16.KL
- net DB4: now also X4-11.KL; no longer X4-17.KL
- net DB5: now also X4-12.KL; no longer X4-18.KL
- net DB6: now also X4-13.KL; no longer X4-19.KL
- net DB7: now also X4-14.KL; no longer X4-20.KL
- net GND: no longer X4-37.KL
- net LCD_NRD: now also X4-17.KL
- net LCD_NRESET: now also X4-18.KL
- net RX1: now also X4-33.KL; no longer X4-24.KL
- net SWCLK: now also X4-37.KL; no longer X4-26.KL
- net SWDIO: now also X4-36.KL; no longer X4-25.KL
- net TESTSIG: now also X4-30.KL; no longer X4-8.KL
- net TL_PWM: now also X4-15.KL; no longer X4-21.KL
- net TRIG: now also X4-31.KL; no longer X4-7.KL
- net TX1: now also X4-32.KL; no longer X4-23.KL
- net USBDM: now also X4-34.KL
- net USBDP: now also X4-35.KL
- net V-MON: now also X4-29.KL; no longer X4-9.KL
- net VGEN: now also X4-16.KL; no longer X4-22.KL
- net VSENSEL1: no longer X4-13.KL
- net VSENSEL2: no longer X4-14.KL
